File: encoder.sch (KiCad schematic (older format))
At the start: 35 parts

Commit message: several enhancements
Parts:
- removed E?: Encoder2, symbol Encoder2
- removed E?: Walter_Encoder_fixed, symbol Walter_Encoder_fixed
- added E2: Encoder2, symbol Encoder2
- added E5: Walter_Encoder_fixed, symbol Walter_Encoder_fixed
- gave numbers to parts that had none: 33
Connections:
- wire segments 67 -> 97
Other:
- note added: "1"
- note added: "2"
- note added: "3"
- note added: "4"
- note added: "5"
- moved on the sheet: R16
